File: Proyecto_TCE/Eagle/Board_con_antena.brd (EAGLE design)
At the start: 55.7 x 22.9 mm, 54 parts, among them J1 HEADER_3X1, J2 HEADER_16X1, J3 HEADER_16X1, J4 HEADER_3X1, J5 MICROUSB, J6 DEBUG_CONNECTOR, J7 FPC_05P-RA-SMD, J8 MM8130-2600, U1 NRF52832, U2 TLV1117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

Commit message: add Board_con_antena
Routing:
- net N$1: track 1.19 -> 43.0 mm
- net S$1: track 19.5 -> 0.00 mm
- net S$2: track 5.14 -> 0.00 mm
Other:
- board size 55.7 x 22.9 mm -> 59.4 x 22.9 mm
Changed lines of the file:
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@@
 <?xml version="1.0" encoding="utf-8"?>
 <!DOCTYPE eagle SYSTEM "eagle.dtd">
-<eagle version="7.7.0">
+<eagle version="9.6.2">
 <drawing>
 <settings>
 <setting alwaysvectorfont="no"/>
+<setting keepoldvectorfont="yes"/>
 <setting verticaltext="up"/>
 </settings>
@@
 <layer number="25" name="tNames" color="7" fill="1" visible="no" active="yes"/>
 <layer number="26" name="bNames" color="7" fill="1" visible="no" active="yes"/>
-<layer number="27" name="tValues" color="7" fill="1" visible="no" active="yes"/>
+<layer number="27" name="tValues" color="7" fill="1" visible="yes" active="yes"/>
 <layer number="28" name="bValues" color="7" fill="1" visible="no" active="yes"/>
 <layer number="29" name="tStop" color="7" fill="3" visible="yes" active="yes"/>
@@
 Bluetooth Low Energy board</description>
 <plain>
-<wire x1="0" y1="0" x2="55.66" y2="0" width="0" layer="20"/>
-<wire x1="55.66" y1="0" x2="55.66" y2="22.86" width="0" layer="20"/>
-<wire x1="55.66" y1="22.86" x2="0" y2="22.86" width="0" layer="20"/>
+<wire x1="0" y1="0" x2="59.36" y2="0" width="0" layer="20"/>
+<wire x1="59.36" y1="0" x2="59.36" y2="22.86" width="0" layer="20"/>
+<wire x1="59.36" y1="22.86" x2="0" y2="22.86" width="0" layer="20"/>
 <wire x1="0" y1="22.86" x2="0" y2="0" width="0" layer="20"/>
 <rectangle x1="50.94" y1="0" x2="55.74" y2="22.9" layer="41"/>
@@
 <text x="16.51" y="20.32" size="1" layer="21" font="vector" ratio="15" rot="R270" align="center-left">4</text>
 <rectangle x1="49.4" y1="9.3" x2="50.9" y2="11.7" layer="41"/>
+<dimension x1="52.05199375" y1="10.7311625" x2="50.85199375" y2="10.86945625" x3="51.45199375" y3="-9.12175" textsize="1" layer="1" dtype="horizontal" visible="yes"/>
+<dimension x1="58.45199375" y1="15.845425" x2="58.193409375" y2="5.845425" x3="62.013809375" y3="10.845425" textsize="1" layer="1" dtype="vertical" visible="yes"/>
+<dimension x1="52.85199375" y1="9.562575" x2="54.05199375" y2="9.7470625" x3="53.45199375" y3="20.987796875" textsize="1" layer="1" dtype="horizontal" visible="yes"/>
+<dimension x1="54.45199375" y1="6.245425" x2="56.1032875" y2="6.94006875" x3="55.277640625" y3="-1.982878125" textsize="1" layer="1" dtype="horizontal" visible="yes"/>
+<dimension x1="56.25199375" y1="6.03978125" x2="58.85199375" y2="6.3468875" x3="57.55199375" y3="2.6104125" textsize="1" layer="1" dtype="horizontal" visible="yes"/>
+<dimension x1="56.85199375" y1="11.518540625" x2="58.05199375" y2="11.518540625" x3="57.45199375" y3="17.765134375" textsize="1" layer="1" dtype="horizontal" visible="yes"/>
 </plain>
 <attributes>
@@
 <param name="dpMaxLengthDifference" value="10mm"/>
 <param name="dpGapFactor" value="2.5"/>
-<param name="checkGrid" value="0"/>
 <param name="checkAngle" value="0"/>
 <param name="checkFont" value="1"/>
 <param name="checkRestrict" value="1"/>
+<param name="checkStop" value="0"/>
+<param name="checkValues" value="0"/>
+<param name="checkNames" value="1"/>
+<param name="checkWireStubs" value="1"/>
+<param name="checkPolygonWidth" value="0"/>
 <param name="useDiameter" value="13"/>
 <param name="maxErrors" value="50"/>
@@
 <wire x1="49.2" y1="10.85" x2="50.34" y2="10.85" width="0.2" layer="1"/>
 <wire x1="50.34" y1="10.85" x2="50.34" y2="10.8" width="0.2" layer="1"/>
+<wire x1="49.235590625" y1="10.848978125" x2="52.45199375" y2="10.848978125" width="0.8" layer="1"/>
+<wire x1="52.45199375" y1="10.848978125" x2="52.45199375" y2="10.845425" width="0.1524" layer="1"/>
+<wire x1="52.45199375" y1="10.845425" x2="52.45199375" y2="6.245425" width="0.8" layer="1"/>
+<wire x1="52.45199375" y1="6.245425" x2="54.45199375" y2="6.245425" width="0.8" layer="1"/>
+<wire x1="54.45199375" y1="6.245425" x2="54.45199375" y2="15.617390625" width="0.8" layer="1"/>
+<wire x1="54.45199375" y1="15.617390625" x2="56.45199375" y2="15.617390625" width="0.8" layer="1"/>
+<wire x1="56.45199375" y1="15.617390625" x2="56.45199375" y2="6.245425" width="0.8" layer="1"/>
+<wire x1="56.45199375" y1="6.245425" x2="58.45199375" y2="6.245425" width="0.8" layer="1"/>
+<wire x1="58.45199375" y1="6.245425" x2="58.45199375" y2="15.445425" width="0.8" layer="1"/>
+<wire x1="49.235590625" y1="10.848978125" x2="49.2" y2="10.85" width="0" layer="19" extent="1-1"/>
 </signal>
 <signal name="N$2">
@@
 <wire x1="8.9" y1="19.855" x2="8.89" y2="19.865" width="0.4" layer="1"/>
 </signal>
-<signal name="S$1">
-<wire x1="50.343190625" y1="10.808971875" x2="54.743190625" y2="10.808971875" width="0.6" layer="1"/>
-<wire x1="54.743190625" y1="10.808971875" x2="54.743190625" y2="22.008971875" width="0.6" layer="1"/>
-<wire x1="50.920709375" y1="7.224103125" x2="54.7953875" y2="7.20598125" width="0.6" layer="1"/>
-</signal>
-<signal name="S$2">
-<wire x1="54.805959375" y1="7.17988125" x2="54.753765625" y2="12.323278125" width="0.6" layer="1"/>
-</signal>
 </signals>
+<mfgpreviewcolors>
+<mfgpreviewcolor name="soldermaskcolor" color="0xC8008000"/>
+<mfgpreviewcolor name="silkscreencolor" color="0xFFFEFEFE"/>
+<mfgpreviewcolor name="backgroundcolor" color="0xFF282828"/>
+<mfgpreviewcolor name="coppercolor" color="0xFFFFBF00"/>
+<mfgpreviewcolor name="substratecolor" color="0xFF786E46"/>
+</mfgpreviewcolors>
 <errors>
 </errors>
